File: V2L Relay Board/V2L Relay Board.kicad_pcb (KiCad board)
At the start: 2 copper layers, 178 parts, among them IC1 TLV76133DCYR, J10 Screw_Terminal_01x02, J11 Screw_Terminal_01x02, J12 Screw_Terminal_01x02, J19 Screw_Terminal_01x02, J20 Screw_Terminal_01x02, J21 Screw_Terminal_01x02, J22 Screw_Terminal_01x02, J23 Screw_Terminal_01x02, J24 Screw_Terminal_01x02, J25 Screw_Terminal_01x02, J26 Screw_Terminal_01x02, J27 Screw_Terminal_01x02, J28 Screw_Terminal_01x02, J29 Screw_Terminal_01x02, J5 Screw_Terminal_01x02, J6 Screw_Terminal_01x02, J7 Screw_Terminal_01x02, J8 Screw_Terminal_01x02, J9 Screw_Terminal_01x02, K19 G5Q-1A-DC12, K20 G5Q-1A-DC12, K21 G5Q-1A-DC12, K22 G5Q-1A-DC12, K23 G5Q-1A-DC12, K24 G5Q-1A-DC12, K25 G5Q-1A-DC12, K26 G5Q-1A-DC12, K27 G5Q-1A-DC12, K28 G5Q-1A-DC12, K29 G5Q-1A-DC12, K30 G5Q-1A-DC12, K31 G5Q-1A-DC12, K32 G5Q-1A-DC12, K33 G5Q-1A-DC12, K34 G5Q-1A-DC12, Q10 2N7000, Q11 LTV-817C, Q12 LTV-817C, Q13 BC337, Q14 BC337, Q15 2N7000, Q16 2N7000, Q17 2N7000, Q18 2N7000, Q19 LTV-817C, Q20 LTV-817C, Q21 LTV-817C, Q22 LTV-817C, Q23 BC337, Q25 BC337, Q26 2N7000, Q27 BC337, Q28 BC337, Q29 2N7000, Q3 LTV-817C, Q30 2N7000, Q31 2N7000, Q32 LTV-817C, Q33 LTV-817C, Q34 LTV-817C, Q35 LTV-817C, Q40 2N7000, Q41 2N7000, Q42 2N7000, Q43 2N7000, Q44 LTV-817C, Q45 LTV-817C, Q46 LTV-817C, Q47 LTV-817C, Q5 LTV-817C, Q52 BC337, Q53 BC337, Q54 BC337, Q55 BC337, Q56 BC337, Q57 BC337, Q58 BC337, Q59 BC337, Q6 2N7000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

Commit message: Routing iteration 1
Parts:
- moved J19 336.2 mm to (169.5, 63.9)
- moved K20 324.3 mm to (143.7, 52.7), turned to 0 degrees
- moved J5 316.7 mm to (169.5, 153.8)
- moved J20 316.4 mm to (169.5, 81.8)
- moved Q27 308.1 mm to (141.2, 64.8), turned to 180 degrees
- moved R45 304.9 mm to (140.3, 59.5), turned to 0 degrees
- moved K21 303.0 mm to (143.7, 70.6), turned to 0 degrees
- moved D18 302.7 mm to (131.6, 54.5), turned to 0 degrees
- moved S3 300.5 mm to (122.8, 51.2), turned to 180 degrees
- moved K22 298.5 mm to (143.7, 142.7), turned to 0 degrees
- moved R27 297.8 mm to (127.8, 55.3), turned to 0 degrees
- moved Q5 296.7 mm to (131.3, 60.8), turned to 0 degrees
- moved J21 288.3 mm to (169.5, 135.8)
- moved LED2 288.3 mm to (124.0, 62.2)
- moved Q8 288.1 mm to (141.2, 154.9), turned to 180 degrees
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Connections:
- Q10 pad 2: /PB4 -> /PA4
- Q15 pad 2: /PB5 -> /PA5
- Q16 pad 2: /PB8 -> /PA6
- Q17 pad 2: /PB9 -> /PA7
- Q9 pad 2: /PB3 -> /PA11
- U1 pad 11: /PB3 -> unconnected-(U1-PB3-Pad11)
- U1 pad 12: /PB4 -> unconnected-(U1-PB4-Pad12)
- U1 pad 13: /PB5 -> unconnected-(U1-PB5-Pad13)
- U1 pad 16: /PB8 -> unconnected-(U1-PB8-Pad16)
- U1 pad 17: /PB9 -> unconnected-(U1-PB9-Pad17)
- U1 pad 29: unconnected-(U1-PA4-Pad29) -> /PA4
- U1 pad 30: unconnected-(U1-PA5-Pad30) -> /PA5
- U1 pad 31: unconnected-(U1-PA6-Pad31) -> /PA6
- U1 pad 32: unconnected-(U1-PA7-Pad32) -> /PA7
- U1 pad 8: unconnected-(U1-PA11-Pad8) -> /PA11
Routing:
- net /SW_12V: track 0.00 -> 258.1 mm
- net Net-(J25-Pin_1): track 0.00 -> 16.2 mm
- net Net-(J7-Pin_1): track 0.00 -> 16.2 mm
- net Net-(J24-Pin_1): track 0.00 -> 16.2 mm
- net Net-(J22-Pin_1): track 0.00 -> 16.2 mm
- net Net-(J20-Pin_1): track 0.00 -> 16.2 mm
- net Net-(J8-Pin_1): track 0.00 -> 16.2 mm
- net Net-(J29-Pin_1): track 0.00 -> 16.2 mm
- net Net-(J27-Pin_1): track 0.00 -> 16.2 mm
- net Net-(J26-Pin_1): track 0.00 -> 16.2 mm
- net Net-(J6-Pin_1): track 0.00 -> 16.2 mm
- net Net-(J5-Pin_1): track 0.00 -> 16.2 mm
- net Net-(J23-Pin_1): track 0.00 -> 16.2 mm
- net Net-(J21-Pin_1): track 0.00 -> 16.2 mm
- net Net-(J19-Pin_1): track 0.00 -> 16.2 mm
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- added copper zone on In2.Cu, net +12V
- added copper zone on In1.Cu, net GND
Other:
- board outline added: 175.2 x 200.1 mm
- copper layers 2 -> 4
