File: V2L Relay Board/V2L Relay Board.kicad_pcb (KiCad board)
At the start: 4 copper layers, 175.2 x 200.1 mm, 178 parts, among them IC1 TLV76133DCYR, J10 Screw_Terminal_01x02, J11 Screw_Terminal_01x02, J12 Screw_Terminal_01x02, J19 Screw_Terminal_01x02, J20 Screw_Terminal_01x02, J21 Screw_Terminal_01x02, J22 Screw_Terminal_01x02, J23 Screw_Terminal_01x02, J24 Screw_Terminal_01x02, J25 Screw_Terminal_01x02, J26 Screw_Terminal_01x02, J27 Screw_Terminal_01x02, J28 Screw_Terminal_01x02, J29 Screw_Terminal_01x02, J5 Screw_Terminal_01x02, J6 Screw_Terminal_01x02, J7 Screw_Terminal_01x02, J8 Screw_Terminal_01x02, J9 Screw_Terminal_01x02, K19 G5Q-1A-DC12, K20 G5Q-1A-DC12, K21 G5Q-1A-DC12, K22 G5Q-1A-DC12, K23 G5Q-1A-DC12, K24 G5Q-1A-DC12, K25 G5Q-1A-DC12, K26 G5Q-1A-DC12, K27 G5Q-1A-DC12, K28 G5Q-1A-DC12, K29 G5Q-1A-DC12, K30 G5Q-1A-DC12, K31 G5Q-1A-DC12, K32 G5Q-1A-DC12, K33 G5Q-1A-DC12, K34 G5Q-1A-DC12, Q10 2N7000, Q11 LTV-817C, Q12 LTV-817C, Q13 BC337, Q14 BC337, Q15 2N7000, Q16 2N7000, Q17 2N7000, Q18 2N7000, Q19 LTV-817C, Q20 LTV-817C, Q21 LTV-817C, Q22 LTV-817C, Q23 BC337, Q25 BC337, Q26 2N7000, Q27 BC337, Q28 BC337, Q29 2N7000, Q3 LTV-817C, Q30 2N7000, Q31 2N7000, Q32 LTV-817C, Q33 LTV-817C, Q34 LTV-817C, Q35 LTV-817C, Q40 2N7000, Q41 2N7000, Q42 2N7000, Q43 2N7000, Q44 LTV-817C, Q45 LTV-817C, Q46 LTV-817C, Q47 LTV-817C, Q5 LTV-817C, Q52 BC337, Q53 BC337, Q54 BC337, Q55 BC337, Q56 BC337, Q57 BC337, Q58 BC337, Q59 BC337, Q6 2N7000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

Commit message: Updated BOM and PCB WIP
Parts:
- J10, J19, J20, J21, J22, J23, J24, J25, J26, J27, J28, J29, J5, J6, J7, J8: footprint downloaded_libraries:1729128 -> downloaded_libraries:1902547
- moved D23 285.8 mm to (333.9, -183.4), turned to -90 degrees
- moved Q26 283.5 mm to (321.5, -170.4)
- moved D5 282.7 mm to (333.9, -160.9), turned to -90 degrees
- moved S11 281.9 mm to (328.8, -177.2), turned to 90 degrees
- moved Q55 280.8 mm to (338.5, -170.9), turned to 0 degrees
- moved Q18 280.5 mm to (321.5, -147.9)
- moved D18 279.5 mm to (333.9, -138.4), turned to -90 degrees
- moved K27 279.3 mm to (337.0, -184.8)
- moved S9 278.9 mm to (328.8, -154.7), turned to 90 degrees
- moved Q13 277.7 mm to (338.5, -148.4), turned to 0 degrees
- moved LED10 277.2 mm to (323.8, -165.3)
- moved J24 277.2 mm to (363.8, -169.8)
- moved Q7 277.0 mm to (321.5, -125.4)
- moved Q32 276.8 mm to (331.2, -166.7)
- moved D19 276.4 mm to (333.9, -116.0), turned to -90 degrees
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Routing:
- net /SW_12V: track 258.1 -> 0.00 mm
- net /PA11: track 0.00 -> 85.7 mm
- net /PB12: track 0.00 -> 62.1 mm
- net /PA9: track 0.00 -> 44.2 mm
- net /PB13: track 0.00 -> 42.1 mm
- net /PA8: track 0.00 -> 24.2 mm
- net /PB14: track 0.00 -> 22.2 mm
- net /PB15: track 0.00 -> 10.2 mm
- net Net-(Q57-B): track 0.00 -> 5.81 mm
- net Net-(LED2-K): track 11.2 -> 15.5 mm
- net Net-(LED6-K): track 11.4 -> 15.5 mm
- net Net-(LED7-K): track 11.4 -> 15.5 mm
- net Net-(LED1-K): track 11.4 -> 15.5 mm
- net Net-(LED5-K): track 11.4 -> 15.5 mm
- net Net-(LED4-K): track 11.4 -> 15.5 mm
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
Commit message: Finished routing, few DRC errors left
Parts:
- moved D18 288.9 mm to (123.0, 59.1)
- moved D19 288.9 mm to (123.0, 81.6)
- moved D20 288.9 mm to (123.0, 149.1)
- moved D21 288.9 mm to (123.0, 126.6)
- moved D22 288.9 mm to (123.0, 104.1)
- moved D23 288.9 mm to (123.0, 14.1)
- moved D4 288.9 mm to (123.0, 171.6)
- moved D5 288.9 mm to (123.0, 36.6)
- moved J19 288.9 mm to (152.9, 72.7)
- moved J20 288.9 mm to (152.9, 95.2)
- moved J21 288.9 mm to (152.9, 162.8)
- moved J22 288.9 mm to (152.9, 140.2)
- moved J23 288.9 mm to (152.9, 117.7)
- moved J24 288.9 mm to (152.9, 27.8)
- moved J5 288.9 mm to (152.9, 185.2)
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Routing:
- net /SW_12V: track 0.00 -> 386.5 mm
- net GND: track 0.00 -> 95.7 mm
- net /PA0: track 0.00 -> 90.4 mm
- net /PA1: track 0.00 -> 88.4 mm
- net /PA2: track 0.00 -> 85.5 mm
- net /PA3: track 0.00 -> 85.3 mm
- net /PA4: track 0.00 -> 80.6 mm
- net /PB11: track 0.00 -> 71.8 mm
- net /PA10: track 0.00 -> 63.3 mm
- net /PA5: track 0.00 -> 60.6 mm
- net /PB10: track 0.00 -> 51.9 mm
- net /3V3: track 0.00 -> 49.6 mm
- net /PA6: track 0.00 -> 41.0 mm
- net /PB1: track 0.00 -> 31.9 mm
- net /PA7: track 0.00 -> 21.9 mm
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
Commit message: Added PWR/GND vias and screw terminal input for +12V. Still missing mounting hole. 0 DRC errors.
Connections:
- J12 pad 2: unconnected-(J12-Pin_2-Pad2) -> +12V
Routing:
- net /3V3: track 49.6 -> 115.0 mm
- net GND: track 95.7 -> 39.6 mm, vias 0 -> 4
- net Net-(LED13-K): track 5.55 -> 15.5 mm
- net +12V: vias 0 -> 1
Other:
- board size 175.2 x 200.1 mm -> 155 x 182 mm
Changed lines of the file:
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@@
 			(layers "*.Cu" "*.Mask")
 			(remove_unused_layers no)
-			(net "unconnected-(J12-Pin_2-Pad2)")
+			(net "+12V")
 			(pinfunction "Pin_2_2")
-			(pintype "passive+no_connect")
+			(pintype "passive")
 		)
 		(embedded_fonts no)
@@
 		)
 	)
-	(gr_line
-		(start 0.75 196.95)
-		(end 0.75 -3.05)
-		(stroke
-			(width 0.05)
-			(type default)
-		)
-		(layer "Edge.Cuts")
-	)
-	(gr_line
-		(start 1 -3)
-		(end 176 -3)
-		(stroke
-			(width 0.05)
-			(type default)
-		)
-		(layer "Edge.Cuts")
-	)
-	(gr_line
-		(start 1 -3)
-		(end 176 -3)
-		(stroke
-			(width 0.1)
-			(type default)
-		)
-		(layer "Edge.Cuts")
-	)
-	(gr_line
-		(start 1 197)
-		(end 1 -3)
-		(stroke
-			(width 0.1)
-			(type default)
-		)
-		(layer "Edge.Cuts")
-	)
-	(gr_line
-		(start 176 -3)
-		(end 176 197)
+	(gr_rect
+		(start 11 11)
+		(end 166 193)
 		(stroke
 			(width 0.05)
 			(type default)
 		)
-		(layer "Edge.Cuts")
-	)
-	(gr_line
-		(start 176 -3)
-		(end 176 197)
-		(stroke
-			(width 0.1)
-			(type default)
-		)
-		(layer "Edge.Cuts")
-	)
-	(gr_line
-		(start 176 197)
-		(end 1 197)
-		(stroke
-			(width 0.05)
-			(type default)
-		)
-		(layer "Edge.Cuts")
-	)
-	(gr_line
-		(start 176 197)
-		(end 1 197)
-		(stroke
-			(width 0.1)
-			(type default)
-		)
+		(fill no)
 		(layer "Edge.Cuts")
 	)
@@
 	(segment
 		(start 93.6 148.925)
-		(end 94.325 148.2)
+		(end 94.0125 148.5125)
 		(width 1)
 		(layer "F.Cu")
@@
 	)
 	(segment
+		(start 94.0125 148.5125)
+		(end 94.325 148.2)
+		(width 1)
+		(layer "F.Cu")
+		(net "+12V")
+	)
+	(segment
 		(start 91.7 148.925)
 		(end 93.6 148.925)
@@
 		(net "+12V")
 	)
+	(via micro
+		(at 94.0125 148.5125)
+		(size 0.6)
+		(drill 0.3)
+		(layers "F.Cu" "In2.Cu")
+		(net "+12V")
+	)
 	(segment
 		(start 127.675 189.45)
@@
 	)
 	(segment
-		(start 79.1 133.025)
-		(end 87.1 141.025)
-		(width 0.25)
-		(layer "F.Cu")
-		(net "GND")
-	)
-	(segment
-		(start 96.485 179.12)
+		(start 96.48 179.125)
 		(end 97.105 178.5)
 		(width 0.2)
@@
 	)
 	(segment
-		(start 97.105 178.5)
-		(end 97.105 178.81)
+		(start 88.695 178.5)
+		(end 88.695 178.81)
 		(width 0.2)
 		(layer "F.Cu")
@@
 	)
 	(segment
-		(start 107.725 184.6)
-		(end 102.145 179.02)
+		(start 97.105 178.5)
+		(end 97.105 178.81)
 		(width 0.2)
 		(layer "F.Cu")
@@
 	)
 	(segment
-		(start 87.1 146.1)
-		(end 87.1 141.025)
-		(width 0.25)
-		(layer "F.Cu")
-		(net "GND")
-	)
-	(segment
-		(start 88.695 178.81)
-		(end 89.005 179.12)
-		(width 0.2)
-		(layer "F.Cu")
-		(net "GND")
-	)
-	(segment
-		(start 89.005 179.12)
-		(end 96.485 179.12)
-		(width 0.2)
-		(layer "F.Cu")
-		(net "GND")
-	)
-	(segment
-		(start 67.02 177)
-		(end 82.135 177)
+		(start 92.675 179.125)
+		(end 96.48 179.125)
 		(width 0.2)
 		(layer "F.Cu")
@@
 	)
 	(segment
-		(start 79.1 130.35)
-		(end 79.1 133.025)
-		(width 0.25)
-		(layer "F.Cu")
-		(net "GND")
-	)
-	(segment
-		(start 88.695 178.5)
-		(end 88.695 178.81)
-		(width 0.2)
-		(layer "F.Cu")
-		(net "GND")
-	)
-	(segment
-		(start 102.145 179.02)
-		(end 102.145 178.5)
-		(width 0.2)
-		(layer "F.Cu")
-		(net "GND")
-	)
-	(segment
-		(start 81.31 128.14)
-		(end 79.1 130.35)
+		(start 89.925 146.095)
+		(end 87.105 146.095)
 		(width 0.25)
 		(layer "F.Cu")
@@
 	)
 	(segment
-		(start 89.975 136.805)
-		(end 81.31 128.14)
-		(width 0.25)
+		(start 88.695 178.81)
+		(end 89.01 179.125)
+		(width 0.2)
 		(layer "F.Cu")
 		(net "GND")
@@
 	)
 	(segment
-		(start 82.135 177)
-		(end 83.635 178.5)
-		(width 0.2)
-		(layer "F.Cu")
-		(net "GND")
-	)
-	(segment
 		(start 97.105 178.81)
 		(end 97.415 179.12)
@@
 	(segment
 		(start 94.325 146.095)
-		(end 87.105 146.095)
+		(end 89.925 146.095)
 		(width 0.25)
 		(layer "F.Cu")
@@
 	)
 	(segment
+		(start 89.975 138.925)
+		(end 94.325 143.275)
+		(width 0.2)
+		(layer "F.Cu")
+		(net "GND")
+	)
+	(segment
 		(start 87.105 146.095)
 		(end 87.1 146.1)
@@
 	)
 	(segment
+		(start 94.325 143.275)
+		(end 94.325 146.095)
+		(width 0.2)
+		(layer "F.Cu")
+		(net "GND")
+	)
+	(segment
 		(start 101.525 179.12)
 		(end 102.145 178.5)
@@
 	)
 	(segment
-		(start 110.6 184.6)
-		(end 107.725 184.6)
+		(start 89.01 179.125)
+		(end 92.675 179.125)
 		(width 0.2)
 		(layer "F.Cu")
@@
 		(net "GND")
 	)
-	(segment
-		(start 89.975 138.925)
-		(end 89.975 136.805)
-		(width 0.25)
-		(layer "F.Cu")
+	(via blind
+		(at 92.675 179.125)
+		(size 0.6)
+		(drill 0.3)
+		(layers "F.Cu" "In1.Cu")
+		(net "GND")
+	)
+	(via micro
+		(at 89.925 146.095)
+		(size 0.6)
+		(drill 0.3)
+		(layers "F.Cu" "In1.Cu")
+		(net "GND")
+	)
+	(via micro
+		(at 89.975 138.925)
+		(size 0.6)
+		(drill 0.3)
+		(layers "F.Cu" "In1.Cu")
+		(net "GND")
+	)
+	(via blind
+		(at 87.35 38.1)
+		(size 0.6)
+		(drill 0.3)
+		(layers "F.Cu" "In1.Cu")
 		(net "GND")
 	)
@@
 	)
 	(segment
+		(start 84.9 144.9)
+		(end 87.175 142.625)
+		(width 1)
+		(layer "F.Cu")
+		(net "/3V3")
+	)
+	(segment
 		(start 89.025 138.925)
 		(end 89.025 142.25)
@@
 	)
 	(segment
+		(start 89.3 122.69)
+		(end 89.3 94.75)
+		(width 0.25)
+		(layer "F.Cu")
+		(net "/3V3")
+	)
+	(segment
 		(start 89.025 138.395)
 		(end 89.025 138.925)
@@
 	)
 	(segment
+		(start 89.3 94.75)
+		(end 96.55 87.5)
+		(width 0.25)
+		(layer "F.Cu")
+		(net "/3V3")
+	)
+	(segment
+		(start 81.31 130.68)
+		(end 89.3 122.69)
+		(width 0.25)
+		(layer "F.Cu")
+		(net "/3V3")
+	)
+	(segment
 		(start 89.025 142.25)
 		(end 89.4 142.625)
@@
 	)
 	(segment
+		(start 84.9 150.1)
+		(end 84.9 144.9)
+		(width 1)
+		(layer "F.Cu")
+		(net "/3V3")
+	)
+	(segment
 		(start 95.5 164.54)
 		(end 100.45 164.54)
@@
 	)
 	(segment
+		(start 88.9 151.4)
+		(end 86.2 151.4)
+		(width 1)
+		(layer "F.Cu")
+		(net "/3V3")
+	)
+	(segment
+		(start 89.4 150.9)
+		(end 88.9 151.4)
+		(width 1)
+		(layer "F.Cu")
+		(net "/3V3")
+	)
+	(segment
+		(start 86.2 151.4)
+		(end 84.9 150.1)
+		(width 1)
+		(layer "F.Cu")
+		(net "/3V3")
+	)
+	(segment
 		(start 82 164.55)
 		(end 87 164.55)
@@
 	)
 	(segment
+		(start 89.4 150.9)
+		(end 89.4 162.15)
+		(width 1)
+		(layer "F.Cu")
+		(net "/3V3")
+	)
+	(segment
 		(start 89.4 162.15)
 		(end 87 164.55)
@@
 	(segment
 		(start 89.4 148.925)
-		(end 89.4 162.15)
+		(end 89.4 150.9)
+		(width 1)
+		(layer "F.Cu")
+		(net "/3V3")
+	)
+	(segment
+		(start 87.175 142.625)
+		(end 89.4 142.625)
 		(width 1)
 		(layer "F.Cu")
@@
 	)
 	(segment
+		(start 62.9 66.225)
+		(end 62.9 73.8)
+		(width 0.25)
+		(layer "F.Cu")
+		(net "Net-(LED13-K)")
+	)
+	(segment
+		(start 64.48 64.645)
+		(end 62.9 66.225)
+		(width 0.25)
+		(layer "F.Cu")
+		(net "Net-(LED13-K)")
+	)
+	(segment
 		(start 65.45 59.35)
 		(end 64.48 60.32)
@@
 	)
 	(segment
+		(start 64.48 64.5)
+		(end 64.48 64.645)
+		(width 0.25)
+		(layer "F.Cu")
+		(net "Net-(LED13-K)")
+	)
+	(segment
 		(start 58.8 131.94)
 		(end 61.13 129.61)
@@
 		(polygon
 			(pts
-				(xy 44.25 12) (xy 133.55 12) (xy 133.55 199.447024) (xy 44.25 198.383929)
+				(xy 44.25 12) (xy 133.55 12) (xy 133.655372 193.074013) (xy 44.25 193.126041)
 			)
 		)
@@
 		(polygon
 			(pts
-				(xy 44.95 12) (xy 132.8 12) (xy 132.8 197) (xy 44.95 197)
+				(xy 44.95 12) (xy 132.8 12) (xy 132.8 194) (xy 44.95 194)
 			)
 		)

Commit message: Added I/O net name silkscreen and Block M
Other:
- board text added: "+12V"
- board text added: "COM"
- board text added: "PA0"
- board text added: "PA1"
- board text added: "PA10"
- board text added: "PA11"
- board text added: "PA2"
- board text added: "PA3"
- board text added: "PA4"
- board text added: "PA5"
- board text added: "PA6"
- board text added: "PA7"
- board text added: "PA8"
- board text added: "PA9"
- board text added: "PB0"
- board text added: "PB1"
- board text added: "PB10"
- board text added: "PB11"
- board text added: "PB12"
- board text added: "PB13"
- board text added: "PB14"
- board text added: "PB15"
