File: V2L Relay Board/V2L Relay Board.kicad_sch (KiCad schematic)
At the start: 104 parts, among them IC1 TLV76133DCYR, J1 Screw_Terminal_01x02, J10 Screw_Terminal_01x02, J2 Screw_Terminal_01x05, J3 Screw_Terminal_01x02, J4 Screw_Terminal_01x02, J5 Screw_Terminal_01x02, J6 Screw_Terminal_01x02, J7 Screw_Terminal_01x02, J8 Screw_Terminal_01x02, J9 Screw_Terminal_01x02, K1 G2RL-1A, K2 G2RL-1A, K3 G2RL-1A, K4 G2RL-1A, K5 G2RL-1A, K6 G2RL-1A, K7 G2RL-1A, K8 G2RL-1A, K9 G2RL-1A, Q1 BC337, Q10 2N7000, Q11 LTV-817C, Q12 LTV-817C, Q13 BC337, Q14 BC337, Q15 2N7000, Q16 2N7000, Q17 2N7000, Q18 2N7000, Q19 LTV-817C, Q2 BC337, Q20 LTV-817C, Q21 LTV-817C, Q22 LTV-817C, Q23 BC337, Q24 BC337, Q25 BC337, Q27 2N7000, Q28 LTV-817C, Q3 LTV-817C, Q4 BC337, Q5 LTV-817C, Q6 2N7000, Q7 2N7000, Q8 BC337, Q9 2N7000, U1 YAAJ_BluePill_Part_Like

Commit message: Updated BOM and KiCad files
Parts:
- removed C3, C4, C5, C6: 0.1u, symbol Device:C
- removed D1, D2, D3, D8: 1N4007, Diode_THT:D_DO-41_SOD81_P10.16mm_Horizontal, symbol Diode:1N4007
- removed J1, J3, J4: Screw_Terminal_01x02, symbol Connector:Screw_Terminal_01x02
- removed J2: Screw_Terminal_01x05, symbol Connector:Screw_Terminal_01x05
- removed K1, K2, K3, K4, K5, K6, K7, K8, K9: G2RL-1A, Relay_THT:Relay_SPST_Omron_G2RL-1A, symbol Relay:G2RL-1A
- removed LED9: SML-D12M8WT86, LEDM1620X150N, symbol SML-D12M8WT86:SML-D12M8WT86
- removed Q1, Q2, Q24, Q4: BC337, Package_TO_SOT_THT:TO-92_Inline, symbol Transistor_BJT:BC337
- removed Q27: 2N7000, Package_TO_SOT_THT:TO-92_Inline, symbol Transistor_FET:2N7000
- removed Q28: LTV-817C, DIP762W60P254L460H450Q4N, symbol LTV-817C:LTV-817C
- removed R12: 402, symbol Device:R
- removed R13, R16, R25, R7: 1.8k, symbol Device:R
- removed S10: JS102011CQN, JS102011CQN, symbol JS102011CQN:JS102011CQN
- added C10, C7, C8, C9: 0.1u, downloaded_libraries:CAPC1005X60N, symbol CL05B104KBD6PJC:CL05B104KBD6PJC
- added D18, D19, D20, D21, D22, D23, D24, D25, D26, D27, D28: 1N4007, Diode_THT:D_DO-41_SOD81_P10.16mm_Horizontal, symbol Diode:1N4007
- added J11, J12, J19, J20, J21, J22, J23, J24, J25, J26, J27, J28, J29: Screw_Terminal_01x02, downloaded_libraries:1729128, symbol Connector:Screw_Terminal_01x02
- added K19, K20, K21, K22, K23, K24, K25, K26, K27, K28, K29, K30, K31, K32, K33, K34: G5Q-1A-DC12, downloaded_libraries:G5Q-1A-EL-HA-VH, symbol G5Q-1A-DC12:G5Q-1A-DC12
- added LED10, LED11, LED12, LED13, LED14, LED15, LED16, LED17, LED18: SML-D12M8WT86, downloaded_libraries:LEDM1620X150N, symbol SML-D12M8WT86:SML-D12M8WT86
- added Q26, Q29, Q30, Q31, Q40, Q41, Q42, Q43: 2N7000, Package_TO_SOT_THT:TO-92_Inline, symbol Transistor_FET:2N7000
- added Q27, Q28, Q52, Q53, Q54, Q55, Q56, Q57, Q58, Q59, Q60: BC337, Package_TO_SOT_THT:TO-92_Inline, symbol Transistor_BJT:BC337
- added Q32, Q33, Q34, Q35, Q44, Q45, Q46, Q47: LTV-817C, downloaded_libraries:DIP762W60P254L460H450Q4N, symbol LTV-817C:LTV-817C
- added R28, R29, R30, R31, R36, R37, R38, R39: 430, downloaded_libraries:ERA2AED122X, symbol Device:R
- added R44, R45, R46, R47, R48, R49, R50, R51, R52, R53, R54, R55: 1.8k, downloaded_libraries:ERA6AEB101V, symbol Device:R
- added S11, S12, S13, S14, S15, S16, S17, S18: JS102011CQN, downloaded_libraries:JS102011CQN, symbol JS102011CQN:JS102011CQN
- C1: footprint (none) -> downloaded_libraries:ZRB15x
- C2: footprint (none) -> downloaded_libraries:CAPC0603X35N
- IC1: footprint SOT230P700X180-4N -> downloaded_libraries:SOT230P700X180-4N
- J10, J5, J6, J7, J8, J9: footprint (none) -> downloaded_libraries:1729128
- LED1, LED2, LED3, LED4, LED5, LED6, LED7, LED8: footprint LEDM1620X150N -> downloaded_libraries:LEDM1620X150N
- Q11, Q12, Q19, Q20, Q21, Q22, Q3, Q5: footprint DIP762W60P254L460H450Q4N -> downloaded_libraries:DIP762W60P254L460H450Q4N
- R10, R11, R8, R9: footprint (none) -> Resistor_THT:R_Axial_DIN0207_L6.3mm_D2.5mm_P10.16mm_Horizontal
- R14, R18, R19, R20, R21: value 402 -> 430; footprint (none) -> downloaded_libraries:ERA2AED122X
- R15, R6: value 402 -> 820; footprint (none) -> downloaded_libraries:ERA2AED122X
- R17, R22, R23, R24: footprint (none) -> downloaded_libraries:ERA6AEB101V
- R26: value 402 -> 1k; footprint (none) -> downloaded_libraries:ERA2AED122X
- R27: value 1.8k -> 820; footprint (none) -> downloaded_libraries:ERA2AED122X
- S1, S3, S4, S5, S6, S7, S8, S9: footprint JS102011CQN -> downloaded_libraries:JS102011CQN
- S2: footprint 100SP1T1B4M2QE -> downloaded_libraries:100SP1T1B4M2QE
- U1: footprint (none) -> downloaded_libraries:YAAJ_BluePill_1
Connections:
- net +3.3V is gone; now on net 3V3: R10.2, R11.2, R8.2, R9.2
- net +12V: now also D4.1 (K), D5.1 (K), D6.1 (K), D7.1 (K), D9.1 (K), Q11.4 (COLLECTOR), Q12.4 (COLLECTOR), Q19.4 (COLLECTOR), Q20.4 (COLLECTOR), Q21.4 (COLLECTOR), Q22.4 (COLLECTOR), Q3.4 (COLLECTOR), Q5.4 (COLLECTOR), S2.2, D18.1 (K), D19.1 (K), D20.1 (K), D21.1 (K), D22.1 (K), D23.1 (K), D24.1 (K), D25.1 (K), D26.1 (K), D27.1 (K), D28.1 (K), K19.5 (COIL_2), K20.5 (COIL_2), K21.5 (COIL_2), K22.5 (COIL_2), K23.5 (COIL_2), K24.5 (COIL_2), K25.5 (COIL_2), K26.5 (COIL_2), K27.5 (COIL_2), K28.5 (COIL_2), K29.5 (COIL_2), K30.5 (COIL_2), K31.5 (COIL_2), K32.5 (COIL_2), K33.5 (COIL_2), K34.5 (COIL_2), Q32.4 (COLLECTOR), Q33.4 (COLLECTOR), Q34.4 (COLLECTOR), Q35.4 (COLLECTOR), Q44.4 (COLLECTOR), Q45.4 (COLLECTOR), Q46.4 (COLLECTOR), Q47.4 (COLLECTOR); no longer S2.1
- net 3V3: now also IC1.2 (OUT_1)
- net COM: now also J12.1 (Pin_1)
- net GND: now also S1.3 (NO), S3.3 (NO), S4.3 (NO), S5.3 (NO), S6.3 (NO), S7.3 (NO), S8.3 (NO), S9.3 (NO), C10.1, C7.1, C8.1, C9.1, LED18.1 (K), Q26.1 (S), Q27.3 (E), Q28.3 (E), Q29.1 (S), Q30.1 (S), Q31.1 (S), Q40.1 (S), Q41.1 (S), Q42.1 (S), Q43.1 (S), Q52.3 (E), Q53.3 (E), Q54.3 (E), Q55.3 (E), Q56.3 (E), Q57.3 (E), Q58.3 (E), Q59.3 (E), Q60.3 (E), S11.3 (NO), S12.3 (NO), S13.3 (NO), S14.3 (NO), S15.3 (NO), S16.3 (NO), S17.3 (NO), S18.3 (NO); no longer S1.1 (NC), S3.1 (NC), S4.1 (NC), S5.1 (NC), S6.1 (NC), S7.1 (NC), S8.1 (NC), S9.1 (NC)
- net PA8: now also Q41.2 (G)
- net PB10: now also Q18.2 (G); no longer Q9.2 (G)
- net PB11: now also Q26.2 (G); no longer Q10.2 (G)
- net PB12: now also Q29.2 (G); no longer Q15.2 (G)
- net PB13: now also Q30.2 (G); no longer Q16.2 (G)
- net PB14: now also Q31.2 (G); no longer Q17.2 (G)
- net PB15: now also Q40.2 (G); no longer Q18.2 (G)
- net SW_12V: now also R27.2, S2.3, R28.2, R29.2, R30.2, R31.2, R36.2, R37.2, R38.2, R39.2; no longer S2.2
- net at Q14.1 (C): now also D6.2 (A), K30.1 (COIL_1); no longer D7.2 (A)
- net at Q5.1 (ANODE): now also R27.1
- net at J6.2 (Pin_2): now also K26.3 (NO)
- net at J6.1 (Pin_1): now also K26.2 (COM)
- net at D5.2 (A): now also Q13.1 (C), K26.1 (COIL_1)
- net at D4.2 (A), Q8.1 (C): now also K22.1 (COIL_1)
- net at D9.2 (A), Q25.1 (C): now also K19.1 (COIL_1)
- net at Q25.2 (B): now also R44.2; no longer R27.2
- net at R23.1: now also Q35.3 (EMITTER); no longer Q20.3 (EMITTER)
- net PA3: now reaches J9.1 (Pin_1)
- net PA3: now also R8.1, U1.28 (PA3), C7.2
- net PA2: now reaches J9.2 (Pin_2)
- net PA2: now also R9.1, U1.27 (PA2), C8.2
- net at Q23.1 (C): now also D7.2 (A), K34.1 (COIL_1); no longer D6.2 (A)
- net at R23.2: now also Q14.2 (B); no longer Q23.2 (B)
- net at J10.1 (Pin_1): now also K19.2 (COM)
- net at J10.2 (Pin_2): now also K19.3 (NO)
- net at R26.1: now also LED18.2 (A)
- net at R24.1: now also Q47.3 (EMITTER); no longer Q21.3 (EMITTER)
- net at Q11.3 (EMITTER): now also R44.1
- net at R22.2: now also Q13.2 (B)
- net PB3: now reaches U1.11 (PB3)
- net PB3: now also Q9.2 (G)
- net PB4: now reaches U1.12 (PB4)
- net PB4: now also Q10.2 (G)
- net PB5: now reaches U1.13 (PB5)
- net PB5: now also Q15.2 (G)
- net PB6: now reaches U1.14 (PB6)
- net PB7: now reaches U1.15 (PB7)
- net PB8: now reaches U1.16 (PB8)
- net PB8: now also Q16.2 (G)
- net PB9: now reaches U1.17 (PB9)
- net PB9: now also Q17.2 (G)
- net PA0: now reaches U1.25 (PA0)
- net PA0: now also R11.1, C10.2, J11.2 (Pin_2)
- net PA1: now reaches U1.26 (PA1)
- net PA1: now also R10.1, C9.2, J11.1 (Pin_1)
- net PA9: now reaches U1.6 (PA9)
- net PA9: now also Q42.2 (G)
- net PA10: now reaches U1.7 (PA10)
- net PA10: now also Q43.2 (G)
- net at J5.2 (Pin_2): now also K22.3 (NO)
- net at J5.1 (Pin_1): now also K22.2 (COM)
- net at Q22.3 (EMITTER): now also R22.1
- net at R24.2: now also Q23.2 (B); no longer Q14.2 (B)
- net at Q19.3 (EMITTER): now also R47.1; no longer R22.1
- net at J8.2 (Pin_2): now also K34.3 (NO)
- net at J8.1 (Pin_1): now also K34.2 (COM)
- net at J7.2 (Pin_2): now also K30.3 (NO)
- net at J7.1 (Pin_1): now also K30.2 (COM)
- net at Q5.3 (EMITTER): now also R45.1
- net at Q3.3 (EMITTER): now also R46.1
- net OUT_0: no longer names the net of U1.32 (PA7)
- net OUT_0: no longer R8.1
- net OUT_1: no longer names the net of U1.31 (PA6)
- net OUT_1: no longer R9.1
- net OUT_2: no longer names the net of U1.30 (PA5)
- net OUT_2: no longer R10.1
- net OUT_3: no longer names the net of U1.29 (PA4)
- net OUT_3: no longer R11.1
- new net: Q34.1 (ANODE), R30.1
- new net: D27.2 (A), K32.1 (COIL_1), Q59.1 (C)
- new net: LED15.1 (K), Q41.3 (D), S16.2 (COM)
- new net: LED17.1 (K), Q43.3 (D), S18.2 (COM)
- new net: J24.1 (Pin_1), K27.2 (COM)
- new net: J24.2 (Pin_2), K27.3 (NO)
- new net: D26.2 (A), K31.1 (COIL_1), Q58.1 (C)
- new net: Q58.2 (B), R53.2
- new net: D19.2 (A), K21.1 (COIL_1), Q28.1 (C)
- new net: Q28.2 (B), R46.2
- new net: Q35.1 (ANODE), R31.1
- new net: LED13.2 (A), Q35.2 (CATHODE)
- new net: D20.2 (A), K23.1 (COIL_1), Q52.1 (C)
- new net: Q32.1 (ANODE), R28.1
- new net: LED10.2 (A), Q32.2 (CATHODE)
- new net: Q32.3 (EMITTER), R50.1
- new net: D18.2 (A), K20.1 (COIL_1), Q27.1 (C)
- new net: Q27.2 (B), R45.2
- new net: Q20.3 (EMITTER), R48.1
- new net: Q55.2 (B), R50.2
- new net: LED15.2 (A), Q45.2 (CATHODE)
- new net: J19.1 (Pin_1), K20.2 (COM)
- new net: J19.2 (Pin_2), K20.3 (NO)
- new net: D22.2 (A), K25.1 (COIL_1), Q54.1 (C)
- new net: Q54.2 (B), R49.2
- new net: J25.1 (Pin_1), K28.2 (COM)
- new net: J25.2 (Pin_2), K28.3 (NO)
- new net: D23.2 (A), K27.1 (COIL_1), Q55.1 (C)
- new net: Q34.3 (EMITTER), R52.1
- new net: Q57.2 (B), R52.2
- new net: Q47.1 (ANODE), R39.1
- new net: LED17.2 (A), Q47.2 (CATHODE)
- new net: J28.1 (Pin_1), K32.2 (COM)
- new net: J28.2 (Pin_2), K32.3 (NO)
- new net: D28.2 (A), K33.1 (COIL_1), Q60.1 (C)
- new net: Q33.3 (EMITTER), R51.1
- new net: Q56.2 (B), R51.2
- new net: Q46.1 (ANODE), R38.1
- new net: LED16.2 (A), Q46.2 (CATHODE)
- new net: Q46.3 (EMITTER), R55.1
- new net: Q21.3 (EMITTER), R49.1
- new net: J20.1 (Pin_1), K21.2 (COM)
- new net: J20.2 (Pin_2), K21.3 (NO)
- new net: J26.1 (Pin_1), K29.2 (COM)
- new net: J26.2 (Pin_2), K29.3 (NO)
- new net: Q44.1 (ANODE), R36.1
- new net: Q33.1 (ANODE), R29.1
- new net: LED16.1 (K), Q42.3 (D), S17.2 (COM)
- new net: Q53.2 (B), R48.2
- new net: LED14.2 (A), Q44.2 (CATHODE)
- new net: Q44.3 (EMITTER), R53.1
- new net: LED12.1 (K), Q30.3 (D), S13.2 (COM)
- new net: LED12.2 (A), Q34.2 (CATHODE)
- new net: LED14.1 (K), Q40.3 (D), S15.2 (COM)
- new net: J29.1 (Pin_1), K33.2 (COM)
- new net: J29.2 (Pin_2), K33.3 (NO)
- new net: LED11.2 (A), Q33.2 (CATHODE)
- new net: D21.2 (A), K24.1 (COIL_1), Q53.1 (C)
- new net: LED13.1 (K), Q31.3 (D), S14.2 (COM)
- new net: Q45.3 (EMITTER), R54.1
- new net: Q59.2 (B), R54.2
- new net: D25.2 (A), K29.1 (COIL_1), Q57.1 (C)
- new net: LED10.1 (K), Q26.3 (D), S11.2 (COM)
- new net: Q52.2 (B), R47.2
- new net: LED11.1 (K), Q29.3 (D), S12.2 (COM)
- new net: J27.1 (Pin_1), K31.2 (COM)
- new net: J27.2 (Pin_2), K31.3 (NO)
- new net: J22.1 (Pin_1), K24.2 (COM)
- new net: J22.2 (Pin_2), K24.3 (NO)
- new net: D24.2 (A), K28.1 (COIL_1), Q56.1 (C)
- new net: J21.1 (Pin_1), K23.2 (COM)
- new net: J21.2 (Pin_2), K23.3 (NO)
- new net: Q60.2 (B), R55.2
- new net: J23.1 (Pin_1), K25.2 (COM)
- new net: J23.2 (Pin_2), K25.3 (NO)
- new net: Q45.1 (ANODE), R37.1
- no-connect marks 0 -> 15
Other:
- note added: "COM"
- note added: "PA13, PA14 - programming/debugging PA11, PA12 - USB PB2 - BOOT1 PC13 - onboard LED (status indication/limited drive) PC14, PC15 - idk PB6, PB7 - I2C display"
- note added: "Y"
- moved on the sheet: C1, C2, D4, IC1, J5, LED1, LED2, LED3, LED4, LED5, LED6, LED7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

Commit message: Routing iteration 1
Connections:
- net PA4: now reaches U1.29 (PA4)
- net PA4: now also Q10.2 (G)
- net PA5: now reaches U1.30 (PA5)
- net PA5: now also Q15.2 (G)
- net PA6: now reaches U1.31 (PA6)
- net PA6: now also Q16.2 (G)
- net PA7: now reaches U1.32 (PA7)
- net PA7: now also Q17.2 (G)
- net PA11: now reaches U1.8 (PA11)
- net PA11: now also Q9.2 (G)
- net PB3: no longer names the net of U1.11 (PB3)
- net PB3: no longer Q9.2 (G)
- net PB4: no longer names the net of U1.12 (PB4)
- net PB4: no longer Q10.2 (G)
- net PB5: no longer names the net of U1.13 (PB5)
- net PB5: no longer Q15.2 (G)
- net PB8: no longer names the net of U1.16 (PB8)
- net PB8: no longer Q16.2 (G)
- net PB9: no longer names the net of U1.17 (PB9)
- net PB9: no longer Q17.2 (G)
- no-connect marks 15 -> 16
Changed lines of the file:
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@@
 	)
 	(no_connect
-		(at 198.12 320.04)
+		(at 157.48 342.9)
 	)
 	(no_connect
-		(at 106.68 339.09)
+		(at 198.12 320.04)
 	)
 	(no_connect
-		(at 198.12 335.28)
+		(at 106.68 339.09)
 	)
 	(no_connect
-		(at 198.12 337.82)
+		(at 157.48 350.52)
 	)
 	(no_connect
-		(at 198.12 340.36)
+		(at 157.48 353.06)
 	)
 	(no_connect
@@
 	)
 	(no_connect
-		(at 198.12 360.68)
+		(at 157.48 337.82)
 	)
 	(no_connect
-		(at 198.12 332.74)
+		(at 157.48 340.36)
+	)
+	(no_connect
+		(at 198.12 360.68)
 	)
 	(no_connect
@@
 	)
 	(no_connect
-		(at 157.48 330.2)
+		(at 30.48 275.59)
 	)
 	(wire
@@
 		)
 	)
-	(label "PB4"
+	(label "PA4"
 		(at 21.59 275.59 0)
 		(effects
@@
 		)
 	)
+	(label "PA11"
+		(at 157.48 330.2 0)
+		(effects
+			(font
+				(size 1.27 1.27)
+			)
+			(justify left bottom)
+		)
+	)
 	(label "SW_12V"
 		(at 279.4 95.25 0)
@@
 		)
 	)
+	(label "PA4"
+		(at 198.12 340.36 0)
+		(effects
+			(font
+				(size 1.27 1.27)
+			)
+			(justify left bottom)
+		)
+	)
 	(label "PA1"
 		(at 19.05 373.38 0)
@@
 		)
 	)
-	(label "PA10"
-		(at 157.48 327.66 0)
+	(label "PA6"
+		(at 198.12 335.28 0)
 		(effects
 			(font
@@
 		)
 	)
-	(label "PB4"
-		(at 157.48 340.36 0)
+	(label "PA10"
+		(at 157.48 327.66 0)
 		(effects
 			(font
@@
 		)
 	)
-	(label "PB5"
-		(at 157.48 342.9 0)
-		(effects
-			(font
-				(size 1.27 1.27)
-			)
-			(justify left bottom)
-		)
-	)
 	(label "PB13"
 		(at 157.48 314.96 0)
@@
 		)
 	)
-	(label "PB5"
+	(label "PA5"
 		(at 144.78 69.85 0)
 		(effects
@@
 		)
 	)
-	(label "PB3"
+	(label "PA11"
 		(at 21.59 207.01 0)
 		(effects
@@
 		)
 	)
-	(label "PB3"
-		(at 157.48 337.82 0)
-		(effects
-			(font
-				(size 1.27 1.27)
-			)
-			(justify left bottom)
-		)
-	)
 	(label "PB14"
 		(at 267.97 275.59 0)
@@
 		)
 	)
-	(label "PB8"
-		(at 157.48 350.52 0)
-		(effects
-			(font
-				(size 1.27 1.27)
-			)
-			(justify left bottom)
-		)
-	)
 	(label "SW_12V"
 		(at 156.21 26.67 0)
@@
 		)
 	)
-	(label "PB9"
-		(at 144.78 207.01 0)
+	(label "PA9"
+		(at 157.48 325.12 0)
 		(effects
 			(font
@@
 		)
 	)
-	(label "PA9"
-		(at 157.48 325.12 0)
+	(label "PA7"
+		(at 198.12 332.74 0)
 		(effects
 			(font
@@
 		)
 	)
-	(label "PB8"
+	(label "PA6"
 		(at 144.78 138.43 0)
 		(effects
@@
 		)
 	)
+	(label "PA5"
+		(at 198.12 337.82 0)
+		(effects
+			(font
+				(size 1.27 1.27)
+			)
+			(justify left bottom)
+		)
+	)
 	(label "SW_12V"
 		(at 33.02 163.83 0)
@@
 		)
 	)
+	(label "PA7"
+		(at 144.78 207.01 0)
+		(effects
+			(font
+				(size 1.27 1.27)
+			)
+			(justify left bottom)
+		)
+	)
 	(label "PA1"
 		(at 73.66 375.92 0)
@@
 		(effects
 			(font
-				(size 1.27 1.27)
-			)
-			(justify left bottom)
-		)
-	)
-	(label "PB9"
-		(at 157.48 353.06 0)
-		(effects
-			(font

Commit message: Updated BOM and PCB WIP
Parts:
- J10, J19, J20, J21, J22, J23, J24, J25, J26, J27, J28, J29, J5, J6, J7, J8: footprint downloaded_libraries:1729128 -> downloaded_libraries:1902547
Changed lines of the file:
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@@
 			)
 		)
-		(property "Footprint" "downloaded_libraries:1729128"
+		(property "Footprint" "downloaded_libraries:1902547"
 			(at 363.22 27.94 0)
 			(hide yes)
@@
 			)
 		)
-		(property "Footprint" "downloaded_libraries:1729128"
+		(property "Footprint" "downloaded_libraries:1902547"
 			(at 363.22 96.52 0)
 			(hide yes)
@@
 			)
 		)
-		(property "Footprint" "downloaded_libraries:1729128"
+		(property "Footprint" "downloaded_libraries:1902547"
 			(at 486.41 96.52 0)
 			(hide yes)
@@
 			)
 		)
-		(property "Footprint" "downloaded_libraries:1729128"
+		(property "Footprint" "downloaded_libraries:1902547"
 			(at 116.84 27.94 0)
 			(hide yes)
@@
 			)
 		)
-		(property "Footprint" "downloaded_libraries:1729128"
+		(property "Footprint" "downloaded_libraries:1902547"
 			(at 363.22 233.68 0)
 			(hide yes)
@@
 			)
 		)
-		(property "Footprint" "downloaded_libraries:1729128"
+		(property "Footprint" "downloaded_libraries:1902547"
 			(at 363.22 165.1 0)
 			(hide yes)
@@
 			)
 		)
-		(property "Footprint" "downloaded_libraries:1729128"
+		(property "Footprint" "downloaded_libraries:1902547"
 			(at 486.41 165.1 0)
 			(hide yes)
@@
 			)
 		)
-		(property "Footprint" "downloaded_libraries:1729128"
+		(property "Footprint" "downloaded_libraries:1902547"
 			(at 240.03 96.52 0)
 			(hide yes)
@@
 			)
 		)
-		(property "Footprint" "downloaded_libraries:1729128"
+		(property "Footprint" "downloaded_libraries:1902547"
 			(at 116.84 165.1 0)
 			(hide yes)
@@
 			)
 		)
-		(property "Footprint" "downloaded_libraries:1729128"
+		(property "Footprint" "downloaded_libraries:1902547"
 			(at 240.03 233.68 0)
 			(hide yes)
@@
 			)
 		)
-		(property "Footprint" "downloaded_libraries:1729128"
+		(property "Footprint" "downloaded_libraries:1902547"
 			(at 240.03 27.94 0)
 			(hide yes)
@@
 			)
 		)
-		(property "Footprint" "downloaded_libraries:1729128"
+		(property "Footprint" "downloaded_libraries:1902547"
 			(at 116.84 96.52 0)
 			(hide yes)
@@
 			)
 		)
-		(property "Footprint" "downloaded_libraries:1729128"
+		(property "Footprint" "downloaded_libraries:1902547"
 			(at 486.41 27.94 0)
 			(hide yes)
@@
 			)
 		)
-		(property "Footprint" "downloaded_libraries:1729128"
+		(property "Footprint" "downloaded_libraries:1902547"
 			(at 486.41 233.68 0)
 			(hide yes)
@@
 			)
 		)
-		(property "Footprint" "downloaded_libraries:1729128"
+		(property "Footprint" "downloaded_libraries:1902547"
 			(at 116.84 233.68 0)
 			(hide yes)
@@
 			)
 		)
-		(property "Footprint" "downloaded_libraries:1729128"
+		(property "Footprint" "downloaded_libraries:1902547"
 			(at 240.03 165.1 0)
 			(hide yes)

Commit message: Added PWR/GND vias and screw terminal input for +12V. Still missing mounting hole. 0 DRC errors.
Connections:
- net +12V: now also J12.2 (Pin_2)
- no-connect marks 16 -> 15
Other:
- note removed: "COM"
Changed lines of the file:
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@@
 		)
 	)
-	(text "COM"
-		(exclude_from_sim no)
-		(at 16.51 378.714 0)
-		(effects
-			(font
-				(size 1.27 1.27)
-			)
-		)
-	)
 	(text "Y"
 		(exclude_from_sim no)
@@
 	)
 	(no_connect
-		(at 21.59 381)
-	)
-	(no_connect
 		(at 198.12 355.6)
 	)
@@
 	(wire
 		(pts
+			(xy 16.51 381) (xy 21.59 381)
+		)
+		(stroke
+			(width 0)
+			(type default)
+		)
+	)
+	(wire
+		(pts
 			(xy 201.93 237.49) (xy 201.93 231.14)
 		)
@@
 		(effects
 			(font
+				(size 1.27 1.27)
+			)
+			(justify left bottom)
+		)
+	)
+	(label "+12V"
+		(at 16.51 381 0)
+		(effects
+			(font
